File: projects/PROTO0001/PROTO0001.sch (EAGLE design)
At the start: 10 parts, among them U1 PIC24FJ256GB406

Commit message: Added i2c peripherals (accelerometer and HR/oximeter)
Parts:
- added C10: CAP_1U_0603_CERAMIC, CattleFit:CAP_1U_0603_CERAMIC
- added C7: CAP_100N_0402_CERAMIC, CattleFit:CAP_100N_0402_CERAMIC
- added C8: CAP_4.7U_0603_CERAMIC, CattleFit:CAP_4.7U_0603_CERAMIC
- added C9: CAP_10U_0805_CERAMIC, CattleFit:CAP_10U_0805_CERAMIC
- added J1: HEADER_2.54MM_1X6, CattleFit:HEADER_2.54MM_1X6
- added R3, R4, R5: (no value), CattleFit:RES_4.7K_0402
- added U2: MMA8452Q, CattleFit:MMA8452Q
- added U3: MAX30100, CattleFit:MAX30100
- C5: value CAP_100N_0402_CERAMIC -> CAP_10U_0805_CERAMIC; device CattleFit:CAP_100N_0402_CERAMIC -> CattleFit:CAP_10U_0805_CERAMIC
Connections:
- removed net MCU_AVDD: C6.1, U1.AVDD
- removed net MCU_AVSS: C6.2, U1.AVSS
- removed net MCU_VDD: C2.1, C3.1, U1.VDD
- new net !HR_INT: R5.1, U3.!INT
- new net 1V8: C10.1, U3.VDD
- new net 3V3: C9.1, U3.IR_LED+, U3.R_LED+
- new net 5V0: C2.1, C3.1, C6.1, C7.1, C8.1, R3.2, R4.2, R5.2, U1.AVDD, U1.VBAT, U1.VDD, U2.VDD, U2.VDDIO
- new net ACC_INT1: U2.INT1
- new net ACC_INT2: U2.INT2
- new net I2C_SCL: R3.1, U1.RE7, U2.SCL, U3.SCL
- new net I2C_SDA: R4.1, U1.RE6, U2.SDA, U3.SDA
- new net PGEC: J1.5, U1.RB1
- new net PGED: J1.4, U1.RB0
- new net VUNREGULATED: J1.2
- net GND: now also C10.2, C2.2, C3.2, C4.2, C6.2, C7.2, C8.2, C9.2, J1.3, S1.S, U1.AVSS, U1.VSS, U2.GND, U2.SA0, U3.GND, U3.PGND
- net MCU_VSS: no longer C2.2, C3.2, C4.2, U1.VSS
- net N$1: now also U2.BYP; no longer S1.S
- net N$2: now also J1.1
Other:
- note added: "5V0 from ICSP"
- note added: "Accelerometer"
- note added: "Addr: 0x1C (SA = 0), 0x1D (SA = 1)"
- note added: "Heart Rate/Oximetry"
- note added: "ICSP Header"
- note added: "Pullup values may need to be changed...330?"
